File: MiteOut_Rohith's_version/ADC.kicad_sch (KiCad schematic)
At the start: 18 parts, among them J3 Screw_Terminal_01x06, Q1 SS8550, SW1 SW_SPDT, U11 HX711

Commit message: Full Schematic Draft 1
Connections:
- net RATE renamed Rate
- net SCLK renamed SCK
Changed lines of the file:
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@@
 		)
 	)
-	(global_label "DataOut"
+	(hierarchical_label "Rate"
 		(shape input)
-		(at 175.26 91.44 0)
-		(fields_autoplaced yes)
+		(at 168.91 124.46 0)
 		(effects
 			(font
@@
 			(justify left)
 		)
-		(property "Intersheetrefs" "${INTERSHEET_REFS}"
-			(at 185.7441 91.44 0)
-			(hide yes)
-			(show_name no)
-			(do_not_autoplace no)
-			(effects
-				(font
-					(size 1.27 1.27)
-				)
-				(justify left)
-			)
-		)
 	)
-	(global_label "SCLK"
+	(hierarchical_label "SCK"
 		(shape input)
 		(at 175.26 95.25 0)
-		(fields_autoplaced yes)
 		(effects
 			(font
@@
 			(justify left)
 		)
-		(property "Intersheetrefs" "${INTERSHEET_REFS}"
-			(at 183.0228 95.25 0)
-			(hide yes)
-			(show_name no)
-			(do_not_autoplace no)
-			(effects
-				(font
-					(size 1.27 1.27)
-				)
-				(justify left)
-			)
-		)
 	)
-	(global_label "RATE"
+	(hierarchical_label "DataOut"
 		(shape input)
-		(at 168.91 124.46 0)
-		(fields_autoplaced yes)
+		(at 175.26 91.44 0)
 		(effects
 			(font
@@
 			(justify left)
 		)
-		(property "Intersheetrefs" "${INTERSHEET_REFS}"
-			(at 176.3704 124.46 0)
-			(hide yes)
-			(show_name no)
-			(do_not_autoplace no)
-			(effects
-				(font
-					(size 1.27 1.27)
-				)
-				(justify left)
-			)
-		)
 	)

Commit message: some error fixes
Connections:
- net at Q1.1 (B): now also U11.2 (BASE)
Changed lines of the file:
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@@
+	(wire
+		(pts
+			(xy 137.16 77.47) (xy 137.16 87.63)
+		)
+		(stroke
+			(width 0)
+			(type default)
+		)
+	)
 	(wire
 		(pts
@@
 	(wire
 		(pts
+			(xy 135.89 77.47) (xy 137.16 77.47)
+		)
+		(stroke
+			(width 0)
+			(type default)
+		)
+	)
+	(wire
+		(pts
 			(xy 119.38 99.06) (xy 115.57 99.06)
 		)
@@
 		)
 		(stroke
+			(width 0)
+			(type default)
+		)
+	)
+	(wire
+		(pts
+			(xy 137.16 87.63) (xy 142.24 87.63)
+		)
+		(stroke

Commit message: Fully checked schematic
Connections:
- net Rate renamed rate
Other:
- note added: "no screw terminal JST/Micro JST"
- note added: "possibly 2 for mic or loadcell+mic on single board"
Changed lines of the file:
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@@
 	(generator_version "10.0")
 	(paper "A4")
+	(text "no screw terminal JST/Micro JST"
+		(exclude_from_sim no)
+		(at 80.518 110.744 0)
+		(effects
+			(font
+				(size 1.27 1.27)
+			)
+		)
+	)
+	(text "possibly 2 for mic or loadcell+mic on single board\n"
+		(exclude_from_sim no)
+		(at 229.362 90.678 0)
+		(effects
+			(font
+				(size 1.27 1.27)
+			)
+		)
+	)
 	(junction
 		(at 132.08 119.38)
@@
 	)
 	(junction
+		(at 157.48 76.2)
+		(diameter 0)
+		(color 0 0 0 0)
+	)
+	(junction
 		(at 168.91 110.49)
 		(diameter 0)
@@
 	)
 	(junction
-		(at 157.48 76.2)
-		(diameter 0)
-		(color 0 0 0 0)
-	)
-	(junction
 		(at 129.54 101.6)
 		(diameter 0)
@@
 	(wire
 		(pts
+			(xy 157.48 68.58) (xy 157.48 76.2)
+		)
+		(stroke
+			(width 0)
+			(type default)
+		)
+	)
+	(wire
+		(pts
 			(xy 137.16 87.63) (xy 142.24 87.63)
 		)
@@
 		)
 	)
-	(wire
-		(pts
-			(xy 157.48 72.39) (xy 157.48 76.2)
-		)
-		(stroke
-			(width 0)
-			(type default)
-		)
-	)
-	(hierarchical_label "Rate"
+	(label "rate"
+		(at 168.91 124.46 0)
+		(effects
+			(font
+				(size 1.27 1.27)
+			)
+			(justify left bottom)
+		)
+	)
+	(hierarchical_label "VDDIO"
 		(shape input)
-		(at 168.91 124.46 0)
+		(at 157.48 68.58 0)
 		(effects
 			(font
@@
 					(unit 1)
 				)
-			)
-		)
-	)
-	(symbol
-		(lib_id "power:+5V")
-		(at 157.48 72.39 0)
-		(unit 1)
-		(body_style 1)
-		(exclude_from_sim no)
-		(in_bom yes)
-		(on_board yes)
-		(in_pos_files yes)
-		(dnp no)
-		(fields_autoplaced yes)
-		(property "Reference" "#PWR016"
-			(at 157.48 76.2 0)
-			(hide yes)
-			(show_name no)
-			(do_not_autoplace no)
-			(effects
-				(font
-					(size 1.27 1.27)
-				)
-			)
-		)
-		(property "Value" "VDDIO"
-			(at 157.48 67.31 0)
-			(show_name no)
-			(do_not_autoplace no)
-			(effects
-				(font
-					(size 1.27 1.27)
-				)
-			)
-		)
-		(property "Footprint" ""
-			(at 157.48 72.39 0)
-			(hide yes)
-			(show_name no)
-			(do_not_autoplace no)
-			(effects
-				(font
-					(size 1.27 1.27)
-				)
-			)
-		)
-		(property "Datasheet" ""
-			(at 157.48 72.39 0)
-			(hide yes)
-			(show_name no)
-			(do_not_autoplace no)
-			(effects
-				(font
-					(size 1.27 1.27)
-				)
-			)
-		)
-		(property "Description" "Power symbol creates a global label with name \"+5V\""
-			(at 157.48 72.39 0)
-			(hide yes)
-			(show_name no)
-			(do_not_autoplace no)
-			(effects
-				(font
-					(size 1.27 1.27)
-				)
-			)
-		)
-		(pin "1"
-		)
-		(instances
-			(project "MiteOut_Rohith's_version"
-				(path "/02ec46d8-9fff-42fd-88ff-c4cb11c6dc1b/0c1926be-fc30-442e-a123-dd1ed96f81be"
-					(reference "#PWR016")
-					(unit 1)
-				)
