File: MiteOut_Rohith's_version/BME_RTC.kicad_sch (KiCad schematic)
At the start: 11 parts, among them J5 Conn_01x04_Socket, J6 Conn_01x04_Socket, J7 Conn_01x04_Socket, J8 Conn_01x04_Socket, SW5 SW_Push, U15 DS3231M

Commit message: some changes ig
Parts:
- J5: value Conn_01x04_Socket -> BME1
- J6: value Conn_01x04_Socket -> BME2
- J7: value Conn_01x04_Socket -> BME3
- J8: value Conn_01x04_Socket -> BME4
Connections:
- net +3.3V: now also J5.4 (Pin_4), J6.4 (Pin_4), J7.4 (Pin_4), J8.4 (Pin_4)
- net Wire0 SDA: now reaches J6.1 (Pin_1)
- net Wire0 SDA: now also J5.1 (Pin_1)
- net Wire0 SCLK: now reaches J6.2 (Pin_2)
- net Wire0 SCLK: now also J5.2 (Pin_2)
- net GND: now reaches J6.3 (Pin_3)
- net GND: now also J5.3 (Pin_3), J7.3 (Pin_3), J8.3 (Pin_3)
- net Wire1 SDA: now reaches J7.1 (Pin_1)
- net Wire1 SDA: now also J8.1 (Pin_1)
- net Wire1 SCLK: now reaches J7.2 (Pin_2)
- net Wire1 SCLK: now also J8.2 (Pin_2)

Commit message: Full Schematic Draft 1
Connections:
- net SCLK renamed RTC_SCLK
- net SDA renamed RTC_SDA
- net Wire0 SCLK renamed BME1SCL
- net BME1SCL: no longer J6.2 (Pin_2)
- net Wire0 SDA renamed BME1SDA
- net BME1SDA: no longer J6.1 (Pin_1)
- net Wire1 SCLK renamed BME3SCL
- net BME3SCL: no longer J8.2 (Pin_2)
- net Wire1 SDA renamed BME3SDA
- net BME3SDA: no longer J8.1 (Pin_1)
- new net BME2SCL: J6.2 (Pin_2)
- new net BME2SDA: J6.1 (Pin_1)
- new net BME4SCL: J8.2 (Pin_2)
- new net BME4SDA: J8.1 (Pin_1)
Changed lines of the file:
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@@
 	(wire
 		(pts
-			(xy 170.18 55.88) (xy 170.18 64.77)
+			(xy 170.18 55.88) (xy 170.18 66.04)
 		)
 		(stroke
@@
 	(wire
 		(pts
-			(xy 132.08 55.88) (xy 132.08 64.77)
+			(xy 132.08 55.88) (xy 132.08 66.04)
 		)
 		(stroke
@@
 	(wire
 		(pts
-			(xy 151.13 55.88) (xy 151.13 64.77)
+			(xy 151.13 55.88) (xy 151.13 66.04)
 		)
 		(stroke
@@
 	(wire
 		(pts
-			(xy 187.96 55.88) (xy 187.96 64.77)
+			(xy 187.96 55.88) (xy 187.96 66.04)
 		)
 		(stroke
@@
 		)
 	)
-	(global_label "Wire1 SDA"
-		(shape input)
-		(at 185.42 66.04 270)
+	(hierarchical_label "BME2SDA"
+		(shape input)
+		(at 148.59 66.04 270)
+		(effects
+			(font
+				(size 1.27 1.27)
+			)
+			(justify right)
+		)
+	)
+	(hierarchical_label "SQW"
+		(shape input)
+		(at 97.79 78.74 0)
+		(effects
+			(font
+				(size 1.27 1.27)
+			)
+			(justify left)
+		)
+	)
+	(hierarchical_label "BME3SDA"
+		(shape input)
+		(at 167.64 66.04 270)
+		(effects
+			(font
+				(size 1.27 1.27)
+			)
+			(justify right)
+		)
+	)
+	(hierarchical_label "BME4SCL"
+		(shape input)
+		(at 187.96 66.04 270)
+		(effects
+			(font
+				(size 1.27 1.27)
+			)
+			(justify right)
+		)
+	)
+	(hierarchical_label "RTC_SCLK"
+		(shape input)
+		(at 39.37 71.12 180)
+		(effects
+			(font
+				(size 1.27 1.27)
+			)
+			(justify right)
+		)
+	)
+	(hierarchical_label "BME2SCL"
+		(shape input)
+		(at 151.13 66.04 270)
 		(fields_autoplaced yes)
 		(effects
@@
 			(justify right)
 		)
-		(property "Intersheetrefs" "${INTERSHEET_REFS}"
-			(at 185.42 78.7014 90)
-			(hide yes)
+		(property "Net Class" ""
+			(at 152.4 66.04 90)
 			(show_name no)
 			(do_not_autoplace no)
@@
 				(font
 					(size 1.27 1.27)
+					(italic yes)
 				)
 				(justify right)
@@
 		)
 	)
-	(global_label "SQW"
-		(shape input)
-		(at 97.79 78.74 0)
-		(fields_autoplaced yes)
-		(effects
-			(font
-				(size 1.27 1.27)
-			)
-			(justify left)
-		)
-		(property "Intersheetrefs" "${INTERSHEET_REFS}"
-			(at 104.7666 78.74 0)
-			(hide yes)
-			(show_name no)
-			(do_not_autoplace no)
-			(effects
-				(font
-					(size 1.27 1.27)
-				)
-				(justify left)
-			)
-		)
-	)
-	(global_label "Wire1 SCLK"
-		(shape input)
-		(at 187.96 64.77 270)
-		(fields_autoplaced yes)
-		(effects
-			(font
-				(size 1.27 1.27)
-			)
-			(justify right)
-		)
-		(property "Intersheetrefs" "${INTERSHEET_REFS}"
-			(at 187.96 78.6409 90)
-			(hide yes)
-			(show_name no)
-			(do_not_autoplace no)
-			(effects
-				(font
-					(size 1.27 1.27)
-				)
-				(justify right)
-			)
-		)
-	)
-	(global_label "Wire0 SDA"
-		(shape input)
-		(at 148.59 66.04 270)
-		(fields_autoplaced yes)
-		(effects
-			(font
-				(size 1.27 1.27)
-			)
-			(justify right)
-		)
-		(property "Intersheetrefs" "${INTERSHEET_REFS}"
-			(at 148.59 78.7014 90)
-			(hide yes)
-			(show_name no)
-			(do_not_autoplace no)
-			(effects
-				(font
-					(size 1.27 1.27)
-				)
-				(justify right)
-			)
-		)
-	)
-	(global_label "Wire1 SDA"
-		(shape input)
-		(at 167.64 66.04 270)
-		(fields_autoplaced yes)
-		(effects
-			(font
-				(size 1.27 1.27)
-			)
-			(justify right)
-		)
-		(property "Intersheetrefs" "${INTERSHEET_REFS}"
-			(at 167.64 78.7014 90)
-			(hide yes)
-			(show_name no)
-			(do_not_autoplace no)
-			(effects
-				(font
-					(size 1.27 1.27)
-				)
-				(justify right)
-			)
-		)
-	)
-	(global_label "Wire0 SCLK"
-		(shape input)
-		(at 132.08 64.77 270)
-		(fields_autoplaced yes)
-		(effects
-			(font
-				(size 1.27 1.27)
-			)
-			(justify right)
-		)
-		(property "Intersheetrefs" "${INTERSHEET_REFS}"
-			(at 132.08 78.6409 90)
-			(hide yes)
-			(show_name no)
-			(do_not_autoplace no)
-			(effects
-				(font
-					(size 1.27 1.27)
-				)
-				(justify right)
-			)
-		)
-	)
-	(global_label "Wire0 SDA"
+	(hierarchical_label "RTC_SDA"
+		(shape input)
+		(at 39.37 74.93 180)
+		(effects
+			(font
+				(size 1.27 1.27)
+			)
+			(justify right)
+		)
+	)
+	(hierarchical_label "BME4SDA"
+		(shape input)
+		(at 185.42 66.04 270)
+		(effects
+			(font
+				(size 1.27 1.27)
+			)
+			(justify right)
+		)
+	)
+	(hierarchical_label "BME1SDA"
 		(shape input)
 		(at 129.54 66.04 270)
-		(fields_autoplaced yes)
-		(effects
-			(font
-				(size 1.27 1.27)
-			)
-			(justify right)
-		)
-		(property "Intersheetrefs" "${INTERSHEET_REFS}"
-			(at 129.54 78.7014 90)
-			(hide yes)
-			(show_name no)
-			(do_not_autoplace no)
-			(effects
-				(font
-					(size 1.27 1.27)
-				)
-				(justify right)
-			)
-		)
-	)
-	(global_label "SCLK"
-		(shape input)
-		(at 39.37 71.12 180)
-		(fields_autoplaced yes)
-		(effects
-			(font
-				(size 1.27 1.27)
-			)
-			(justify right)
-		)
-		(property "Intersheetrefs" "${INTERSHEET_REFS}"
-			(at 31.6072 71.12 0)
-			(hide yes)
-			(show_name no)
-			(do_not_autoplace no)
-			(effects
-				(font
-					(size 1.27 1.27)
-				)
-				(justify right)
-			)
-		)
-	)
-	(global_label "SDA"
-		(shape input)
-		(at 39.37 74.93 180)
-		(fields_autoplaced yes)
-		(effects
-			(font
-				(size 1.27 1.27)
-			)
-			(justify right)
-		)
-		(property "Intersheetrefs" "${INTERSHEET_REFS}"
-			(at 32.8167 74.93 0)
-			(hide yes)
-			(show_name no)
-			(do_not_autoplace no)
-			(effects
-				(font
-					(size 1.27 1.27)
-				)
-				(justify right)
-			)
-		)
-	)
-	(global_label "Wire1 SCLK"
-		(shape input)
-		(at 170.18 64.77 270)
-		(fields_autoplaced yes)
-		(effects
-			(font
-				(size 1.27 1.27)
-			)
-			(justify right)
-		)
-		(property "Intersheetrefs" "${INTERSHEET_REFS}"
-			(at 170.18 78.6409 90)
-			(hide yes)
-			(show_name no)
-			(do_not_autoplace no)
-			(effects
-				(font
-					(size 1.27 1.27)
-				)
-				(justify right)
-			)
-		)
-	)
-	(global_label "Wire0 SCLK"
-		(shape input)
-		(at 151.13 64.77 270)
-		(fields_autoplaced yes)
-		(effects
-			(font
-				(size 1.27 1.27)
-			)
-			(justify right)
-		)
-		(property "Intersheetrefs" "${INTERSHEET_REFS}"
-			(at 151.13 78.6409 90)
-			(hide yes)
-			(show_name no)
-			(do_not_autoplace no)
-			(effects
-				(font
-					(size 1.27 1.27)
-				)
-				(justify right)
-			)
-		)
-	)
+		(effects
+			(font
+				(size 1.27 1.27)
+			)
+			(justify right)
+		)
+	)
+	(hierarchical_label "BME3SCL"
+		(shape input)
+		(at 170.18 66.04 270)
+		(effects
+			(font
+				(size 1.27 1.27)
+			)
+			(justify right)
+		)
+	)
+	(hierarchical_label "BME1SCL"
+		(shape input)
+		(at 132.08 66.04 270)
+		(effects
+			(font
+				(size 1.27 1.27)
+			)
+			(justify right)
+		)
+	)

Commit message: some error fixes
Parts:
- removed R12: 10k, symbol Device:R
- added C15: 104uF, symbol Device:C
- added R13: 10k, symbol Device:R
Connections:
- net +3.3V: now also C15.1, R13.1
- net GND: now also BT1.2 (-), C14.1, SW5.1, U15.10 (GND), U15.11 (GND), U15.12 (GND), U15.13 (GND), U15.5 (GND), U15.6 (GND), U15.7 (GND), U15.8 (GND), U15.9 (GND), C15.2
- net SQW: now reaches U15.3 (~{INT}/SQW)
- net SQW: now also R13.2
- no-connect marks 0 -> 1

Commit message: Fully checked schematic
Connections:
- net SQW renamed sqw
Other:
- moved on the sheet: BT1, C14
Changed lines of the file:
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@@
-	)
-	(junction
-		(at 81.28 60.96)
-		(diameter 0)
-		(color 0 0 0 0)
 	)
 	(junction
@@
 	)
 	(junction
-		(at 72.39 60.96)
+		(at 72.39 58.42)
 		(diameter 0)
 		(color 0 0 0 0)
@@
 	)
 	(junction
+		(at 81.28 58.42)
+		(diameter 0)
+		(color 0 0 0 0)
+	)
+	(junction
 		(at 69.85 63.5)
 		(diameter 0)
@@
 	(wire
 		(pts
-			(xy 90.17 60.96) (xy 90.17 93.98)
-		)
-		(stroke
-			(width 0)
-			(type default)
-		)
-	)
-	(wire
-		(pts
 			(xy 72.39 86.36) (xy 72.39 93.98)
 		)
@@
 	(wire
 		(pts
-			(xy 81.28 53.34) (xy 81.28 60.96)
+			(xy 81.28 50.8) (xy 81.28 58.42)
 		)
 		(stroke
@@
 	(wire
 		(pts
-			(xy 72.39 93.98) (xy 90.17 93.98)
-		)
-		(stroke
-			(width 0)
-			(type default)
-		)
-	)
-	(wire
-		(pts
 			(xy 69.85 63.5) (xy 69.85 64.77)
 		)
@@
 	(wire
 		(pts
-			(xy 72.39 53.34) (xy 72.39 60.96)
+			(xy 72.39 50.8) (xy 72.39 58.42)
 		)
 		(stroke
@@
 	(wire
 		(pts
-			(xy 72.39 60.96) (xy 72.39 66.04)
+			(xy 72.39 58.42) (xy 72.39 66.04)
 		)
 		(stroke
@@
 	(wire
 		(pts
-			(xy 81.28 60.96) (xy 90.17 60.96)
-		)
-		(stroke
-			(width 0)
-			(type default)
-		)
-	)
-	(wire
-		(pts
 			(xy 129.54 55.88) (xy 129.54 66.04)
 		)
@@
 	(wire
 		(pts
-			(xy 72.39 60.96) (xy 73.66 60.96)
+			(xy 72.39 58.42) (xy 73.66 58.42)
 		)
 		(stroke
@@
 	(wire
 		(pts
-			(xy 72.39 53.34) (xy 73.66 53.34)
-		)
-		(stroke
-			(width 0)
-			(type default)
+			(xy 72.39 50.8) (xy 73.66 50.8)
+		)
+		(stroke
+			(width 0)
+			(type default)
+		)
+	)
+	(label "sqw"
+		(at 97.79 78.74 0)
+		(effects
+			(font
+				(size 1.27 1.27)
+			)
+			(justify left bottom)
 		)
 	)
@@
 			)
 			(justify right)
-		)
-	)
-	(hierarchical_label "SQW"
-		(shape input)
-		(at 97.79 78.74 0)
-		(effects
-			(font
-				(size 1.27 1.27)
-			)
-			(justify left)
 		)
 	)
@@
 	)
 	(symbol
+		(lib_id "power:GND")
+		(at 81.28 58.42 0)
+		(unit 1)
+		(body_style 1)
+		(exclude_from_sim no)
+		(in_bom yes)
+		(on_board yes)
+		(in_pos_files yes)
+		(dnp no)
+		(fields_autoplaced yes)
+		(property "Reference" "#PWR091"
+			(at 81.28 64.77 0)
+			(hide yes)
+			(show_name no)
+			(do_not_autoplace no)
+			(effects
+				(font
+					(size 1.27 1.27)
+				)
+			)
+		)
+		(property "Value" "GND"
+			(at 81.28 63.5 0)
+			(show_name no)
+			(do_not_autoplace no)
+			(effects
+				(font
+					(size 1.27 1.27)
+				)
+			)
+		)
+		(property "Footprint" ""
+			(at 81.28 58.42 0)
+			(hide yes)
+			(show_name no)
+			(do_not_autoplace no)
+			(effects
+				(font
+					(size 1.27 1.27)
+				)
+			)
+		)
+		(property "Datasheet" ""
+			(at 81.28 58.42 0)
+			(hide yes)
+			(show_name no)
+			(do_not_autoplace no)
+			(effects
+				(font
+					(size 1.27 1.27)
+				)
+			)
+		)
+		(property "Description" "Power symbol creates a global label with name \"GND\" , ground"
+			(at 81.28 58.42 0)
+			(hide yes)
+			(show_name no)
+			(do_not_autoplace no)
+			(effects
+				(font
+					(size 1.27 1.27)
+				)
+			)
+		)
+		(pin "1"
+		)
+		(instances
+			(project "MiteOut_Rohith's_version"
+				(path "/02ec46d8-9fff-42fd-88ff-c4cb11c6dc1b/7b652e73-6186-4556-9128-d1f2a006792a"
+					(reference "#PWR091")
+					(unit 1)
+				)
+			)
+		)
+	)
+	(symbol
 		(lib_id "Connector:Conn_01x04_Socket")
 		(at 132.08 50.8 90)
@@
 	(symbol
 		(lib_id "Device:C")
-		(at 77.47 60.96 270)
+		(at 77.47 58.42 270)
 		(unit 1)
 		(body_style 1)
@@
 		(dnp no)
 		(property "Reference" "C14"
-			(at 77.47 57.658 90)
+			(at 75.692 55.118 90)
 			(show_name no)
 			(do_not_autoplace no)
@@
 		)
 		(property "Value" "104uF"
-			(at 77.47 64.516 90)
+			(at 76.2 61.976 90)
 			(show_name no)
 			(do_not_autoplace no)
@@
 		)
 		(property "Footprint" ""
-			(at 73.66 61.9252 0)
+			(at 73.66 59.3852 0)
 			(hide yes)
 			(show_name no)
@@
 		)
 		(property "Datasheet" ""
-			(at 77.47 60.96 0)
+			(at 77.47 58.42 0)
 			(hide yes)
 			(show_name no)
@@
 		)
 		(property "Description" "Unpolarized capacitor"
-			(at 77.47 60.96 0)
+			(at 77.47 58.42 0)
 			(hide yes)
 			(show_name no)
@@
 	(symbol
 		(lib_id "Device:Battery_Cell")
-		(at 78.74 53.34 90)
+		(at 78.74 50.8 90)
 		(unit 1)
 		(body_style 1)
@@
 		(fields_autoplaced yes)
 		(property "Reference" "BT1"
+			(at 76.8985 43.18 90)
+			(show_name no)
+			(do_not_autoplace no)
+			(effects
+				(font
+					(size 1.27 1.27)
+				)
+			)
+		)
+		(property "Value" "3V Coin Cell"
 			(at 76.8985 45.72 90)
 			(show_name no)
@@
 			)
 		)
-		(property "Value" "3V Coin Cell"
-			(at 76.8985 48.26 90)
-			(show_name no)
-			(do_not_autoplace no)
-			(effects
-				(font
-					(size 1.27 1.27)
-				)
-			)
-		)
 		(property "Footprint" ""
-			(at 77.216 53.34 90)
+			(at 77.216 50.8 90)
 			(hide yes)
 			(show_name no)
@@
 		)
 		(property "Datasheet" ""
-			(at 77.216 53.34 90)
+			(at 77.216 50.8 90)
 			(hide yes)
 			(show_name no)
@@
 		)
 		(property "Description" "Single-cell battery"
-			(at 78.74 53.34 0)
+			(at 78.74 50.8 0)
 			(hide yes)
 			(show_name no)
@@
 		)
 		(property "Sim.Device" "V"
-			(at 78.74 53.34 0)
+			(at 78.74 50.8 0)
 			(hide yes)
 			(show_name no)
@@
 		)
 		(property "Sim.Type" "DC"
-			(at 78.74 53.34 0)
+			(at 78.74 50.8 0)
 			(hide yes)
 			(show_name no)
@@
 		)
 		(property "Sim.Pins" "1=+ 2=-"
-			(at 78.74 53.34 0)
-			(hide yes)
-			(show_name no)
+			(at 78.74 50.8 0)
+			(hide yes)
+			(show_name no)
