File: MiteOut_Rohith's_version/BME_RTC.kicad_sch (KiCad schematic)
At the start: 12 parts, among them J5 BME1, J6 BME2, J7 BME3, J8 BME4, SW5 SW_Push, U15 DS3231M

Commit message: Final June Push
Other:
- note added: "WE only need 1 pressure reading so only 1 needs to be BME others can be cheaper temp+humidity board"
Changed lines of the file:
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@@
 	(generator_version "10.0")
 	(paper "A4")
+	(text "WE only need 1 pressure reading so only 1 needs to be BME others can be cheaper temp+humidity board\n"
+		(exclude_from_sim no)
+		(at 170.688 92.964 0)
+		(effects
+			(font
+				(size 1.27 1.27)
+			)
+		)
+	)
 	(junction
 		(at 69.85 64.77)
