File: MiteOut_Rohith's_version/MiteOut_Rohith's_version.kicad_sch (KiCad schematic)
At the start: 24 parts, among them J4 USB_C_Receptacle_USB2.0_16P, J9 Conn_01x20_Pin, SW3 SW_Push, SW4 SW_Push, U1 ESP32-S3-WROOM-1, U13 D3V3XA4B10LP, U14 TLV75801PDRV, U16 AMS1117CS-3.3

Commit message: Fully checked schematic
Parts:
- removed C22, C23: 10uF, symbol Device:C
- removed D11: LED, LED_SMD:LED_0603_1608Metric_Pad1.05x0.95mm_HandSolder, symbol Device:LED
- removed R34: 1M, Resistor_SMD:R_0603_1608Metric_Pad0.98x0.95mm_HandSolder, symbol Device:R
- removed R35: 200k, Resistor_SMD:R_0603_1608Metric_Pad0.98x0.95mm_HandSolder, symbol Device:R
- removed R36: 5.1k, symbol Device:R
- removed U14: TLV75801PDRV, Package_SON:WSON-6-1EP_2x2mm_P0.65mm_EP1x1.6mm, symbol Regulator_Linear:TLV75801PDRV
- added SC1: Solar_Cell, symbol Device:Solar_Cell
Connections:
- net 5VUSB is gone; now on net +5V: J4.A4 (VBUS), J4.A9 (VBUS), J4.B4 (VBUS), J4.B9 (VBUS), U13.4, U13.7 (NC)
- net Charging + Current measure/VIN/Solar+: now also SC1.1 (+)
- net GND: now also SC1.2 (-)
Other:
- sheet ADC ports: added VDDIO; removed Rate
- sheet BME+RTC ports: added none; removed SQW
- sheet Charging + Current measure ports: added none; removed VBUS
- note added: "Same as MCU power supply"
- moved on the sheet: C16, C17, C18, C19, C20, J4, J9, R14, R15, SW3, SW4, U1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
