File: MiteOut_Rohith's_version/MiteOut_Rohith's_version.kicad_sch (KiCad schematic)
At the start: 18 parts, among them J4 USB_C_Receptacle_USB2.0_16P, J9 Conn_01x20_Pin, SW3 SW_Push, SW4 SW_Push, U1 ESP32-S3-WROOM-1, U13 D3V3XA4B10LP, U16 AMS1117CS-3.3

Commit message: Final June Push
Connections:
- net Data+: no longer U13.10 (NC)
- no-connect marks 7 -> 8
Changed lines of the file:
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@@
-	)
-	(junction
-		(at 77.47 171.45)
-		(diameter 0)
-		(color 0 0 0 0)
 	)
 	(junction
@@
 	)
 	(no_connect
+		(at 82.55 171.45)
+	)
+	(no_connect
 		(at 107.95 186.69)
 	)
@@
 	(wire
 		(pts
-			(xy 77.47 176.53) (xy 77.47 171.45)
+			(xy 77.47 154.94) (xy 77.47 176.53)
 		)
 		(stroke
@@
 	(wire
 		(pts
-			(xy 77.47 171.45) (xy 82.55 171.45)
-		)
-		(stroke
-			(width 0)
-			(type default)
-		)
-	)
-	(wire
-		(pts
 			(xy 50.8 60.96) (xy 54.61 60.96)
 		)
@@
 		)
 		(stroke
-			(width 0)
-			(type default)
-		)
-	)
-	(wire
-		(pts
-			(xy 77.47 171.45) (xy 77.47 154.94)
-		)
-		(stroke
